File: energy-meter/lcr2.sch (KiCad schematic (older format))
At the start: 8 parts

Commit message: remove two of the opamps
We can measure the voltage without an amplifier so let's do it. The other
was used for the LCR outputs, which we don't have here.
Parts:
- removed C85: 270p, 1%, Capacitor_SMD:C_0603_1608Metric_Pad1.05x0.95mm_HandSolder, symbol Device:C
- removed L5: 470u, Inductor_SMD:L_1210_3225Metric_Pad1.42x2.65mm_HandSolder, symbol Device:L
- removed R92, R93: 1k, 1%, Resistor_SMD:R_0603_1608Metric_Pad1.05x0.95mm_HandSolder, symbol Device:R
Connections:
- net labels removed: OP2_OUT, OP2_OUT_F
- wire segments 24 -> 12
Changed lines of the file:
@@
 Comment4 ""
 $EndDescr
-Text Label 1050 2150 0    50   ~ 0
-OP2_OUT
 Text Label 1050 1100 0    50   ~ 0
 OP1_OUT
@@
 Text Label 2600 1100 2    50   ~ 0
 OP1_OUT_F
-$Comp
-L Device:R R?
-U 1 1 60895BB5
-P 1550 2150
-AR Path="/602A3FC4/60895BB5" Ref="R?"  Part="1"
-AR Path="/60514CC5/60895BB5" Ref="R?"  Part="1"
-AR Path="/60514CC5/6084417D/60895BB5" Ref="R92"  Part="1"
-AR Path="/607B74C2/6084417D/60895BB5" Ref="R92"  Part="1"
-F 0 "R92" V 1343 2150 50  0000 C CNN
-F 1 "1k, 1%" V 1434 2150 50  0000 C CNN
-F 2 "Resistor_SMD:R_0603_1608Metric_Pad1.05x0.95mm_HandSolder" V 1480 2150 50  0001 C CNN
-F 3 "~" H 1550 2150 50  0001 C CNN
-	1    1550 2150
-	0    1    1    0
-$EndComp
-$Comp
-L Device:R R?
-U 1 1 60895BBB
-P 2150 2350
-AR Path="/602A3FC4/60895BBB" Ref="R?"  Part="1"
-AR Path="/60514CC5/60895BBB" Ref="R?"  Part="1"
-AR Path="/60514CC5/6084417D/60895BBB" Ref="R93"  Part="1"
-AR Path="/607B74C2/6084417D/60895BBB" Ref="R93"  Part="1"
-F 0 "R93" V 1943 2350 50  0000 C CNN
-F 1 "1k, 1%" V 2034 2350 50  0000 C CNN
-F 2 "Resistor_SMD:R_0603_1608Metric_Pad1.05x0.95mm_HandSolder" V 2080 2350 50  0001 C CNN
-F 3 "~" H 2150 2350 50  0001 C CNN
-	1    2150 2350
-	-1   0    0    1
-$EndComp
-Wire Wire Line
-	1050 2150 1400 2150
-$Comp
-L Device:C C?
-U 1 1 60895BC2
-P 1750 2350
-AR Path="/602A2F7F/60895BC2" Ref="C?"  Part="1"
-AR Path="/602A3FC4/60895BC2" Ref="C?"  Part="1"
-AR Path="/60514CC5/60895BC2" Ref="C?"  Part="1"
-AR Path="/60514CC5/6084417D/60895BC2" Ref="C85"  Part="1"
-AR Path="/607B74C2/6084417D/60895BC2" Ref="C85"  Part="1"
-F 0 "C85" H 1865 2396 50  0000 L CNN
-F 1 "270p, 1%" H 1865 2305 50  0000 L CNN
-F 2 "Capacitor_SMD:C_0603_1608Metric_Pad1.05x0.95mm_HandSolder" H 1788 2200 50  0001 C CNN
-F 3 "~" H 1750 2350 50  0001 C CNN
-	1    1750 2350
-	-1   0    0    -1
-$EndComp
-$Comp
-L Device:L L?
-U 1 1 60895BC9
-P 1950 2150
-AR Path="/60514CC5/60895BC9" Ref="L?"  Part="1"
-AR Path="/60514CC5/6084417D/60895BC9" Ref="L5"  Part="1"
-AR Path="/607B74C2/6084417D/60895BC9" Ref="L5"  Part="1"
-F 0 "L5" V 2140 2150 50  0000 C CNN
-F 1 "470u" V 2049 2150 50  0000 C CNN
-F 2 "Inductor_SMD:L_1210_3225Metric_Pad1.42x2.65mm_HandSolder" H 1950 2150 50  0001 C CNN
-F 3 "~" H 1950 2150 50  0001 C CNN
-F 4 "C295109, C89021" V 1950 2150 50  0001 C CNN "LCSC"
-	1    1950 2150
-	0    -1   -1   0
-$EndComp
-Wire Wire Line
-	2150 2500 2150 2550
-Wire Wire Line
-	2150 2550 1950 2550
-Wire Wire Line
-	1750 2550 1750 2500
-Wire Wire Line
-	1750 2200 1750 2150
-Wire Wire Line
-	1750 2150 1700 2150
-Wire Wire Line
-	1750 2150 1800 2150
-Connection ~ 1750 2150
-Wire Wire Line
-	2100 2150 2150 2150
-Wire Wire Line
-	2150 2150 2150 2200
-$Comp
-L power:GND #PWR?
-U 1 1 60895BD8
-P 1950 2600
-AR Path="/602A2F7F/60895BD8" Ref="#PWR?"  Part="1"
-AR Path="/602A3FC4/60895BD8" Ref="#PWR?"  Part="1"
-AR Path="/60514CC5/60895BD8" Ref="#PWR?"  Part="1"
-AR Path="/60514CC5/6084417D/60895BD8" Ref="#PWR0238"  Part="1"
-AR Path="/607B74C2/6084417D/60895BD8" Ref="#PWR0142"  Part="1"
-F 0 "#PWR0142" H 1950 2350 50  0001 C CNN
-F 1 "GND" V 1955 2472 50  0000 R CNN
-F 2 "" H 1950 2600 50  0001 C CNN
-F 3 "" H 1950 2600 50  0001 C CNN
-	1    1950 2600
-	1    0    0    -1
-$EndComp
-Wire Wire Line
-	1950 2600 1950 2550
-Connection ~ 1950 2550
-Wire Wire Line
-	1950 2550 1750 2550
-Wire Wire Line
-	2150 2150 2600 2150
-Connection ~ 2150 2150
-Text Label 2600 2150 2    50   ~ 0
-OP2_OUT_F
 Text HLabel 1050 1100 0    50   Input ~ 0
 OP1_OUT
-Text HLabel 1050 2150 0    50   Input ~ 0
-OP2_OUT
-Text HLabel 2600 2150 2    50   Input ~ 0
-OP2_OUT_F
 Text HLabel 2600 1100 2    50   Input ~ 0
 OP1_OUT_F
